File: first keyboard.kicad_sch (KiCad schematic)
At the start: 0 parts

Commit message: MCU schematic
Parts:
- added C1: C_Small, symbol Device:C_Small
- added C2, C3, C4: 0.1 uF, symbol Device:C_Small
- added C5: 10 uF, symbol Device:C_Small
- added C6, C7: 22 pF, symbol Device:C_Small
- added F1: 500mA, symbol Device:Polyfuse_Small
- added R1: 10k, symbol Device:R_Small
- added R2, R3: 22, symbol Device:R_Small
- added R4: R_Small, symbol Device:R_Small
- added SW1: SW_Push, symbol Switch:SW_Push
- added U1: ATmega32U4-A, Package_QFP:TQFP-44_10x10mm_P0.8mm, symbol MCU_Microchip_ATmega:ATmega32U4-A
- added USB1: Molex-0548190589, symbol random-keyboard-parts:Molex-0548190589
- added Y1: 16MHz, symbol Device:Crystal_GND24_Small
Connections:
- new net: C7.2, U1.16 (XTAL2), Y1.3
- new net: R4.2, SW1.2, U1.13 (~{RESET})
- new net: R2.1, U1.4 (D+)
- new net: R1.1, U1.33 (~{HWB}/PE2)
- new net: C6.2, U1.17 (XTAL1), Y1.1
- new net: C1.1, U1.6 (UCAP)
- new net: R3.1, U1.3 (D-)
- new net +5V: C2.1, C3.1, C4.1, C5.1, F1.1, R4.1, U1.14 (VCC), U1.2 (UVCC), U1.24 (AVCC), U1.34 (VCC), U1.44 (AVCC), U1.7 (VBUS)
- new net D+: R2.2, USB1.3 (D+)
- new net D-: R3.2, USB1.4 (D-)
- new net GND: C1.2, C2.2, C3.2, C4.2, C5.2, C6.1, C7.1, R1.2, SW1.1, U1.15 (GND), U1.23 (GND), U1.35 (GND), U1.43 (GND), U1.5 (UGND), USB1.1 (GND), Y1.2, Y1.4
- new net VCC: F1.2, USB1.5 (VBUS)
